Commit message: Third commit: Optimize URDF for active Joints 1,3,5 and add real driver with stiction compensation

File: urdf/finger.urdf (robot description, URDF)
Before this commit: robot virtual_finger, 6 links, 5 joints
Links:
- removed link link4
- removed link link5
Joints:
- removed joint joint2
- removed joint joint4
- joint joint3: child link3 -> link2; origin xyz=0 0 0.08 rpy=0 0 0 -> xyz=0 0 0.1 rpy=0 0 0; parent link2 -> link1
- joint joint5: child link5 -> link3; origin xyz=0 0 0.05 rpy=0 0 0 -> xyz=0 0 0.08 rpy=0 0 0; parent link4 -> link2

Commit message: 6th commit: Tune PID gains, set joint offsets, and add protection for faulty joint 3

File: urdf/finger.urdf (robot description, URDF)
Before this commit: robot real_3axis_finger_135, 4 links, 3 joints
Joints:
- joint joint1: limit lower=-1.57 upper=1.57 effort=10 velocity=3.0 -> lower=-3.0 upper=0.5 effort=10 velocity=3.0
